File: Sleepduino/Sleepduino.kicad_pcb (KiCad board)
At the start: 2 copper layers, 93.8 x 119.5 mm, 5 parts, among them J1 USB_B_Micro, U1 ATmega328P-A, Y1 Crystal

Commit message: Updates
Parts:
- added C3: C, Capacitor_SMD:C_0402_1005Metric, F.Cu at (159.3, 106.5)
- added C4: C, Capacitor_SMD:C_0402_1005Metric, F.Cu at (166.9, 106.5)
- added G***: LOGO, Sleepduino:George2, F.Cu at (163.1, 87.4)
- added J2: Conn_02x03_Counter_Clockwise_MountingPin, Connector_PinHeader_2.00mm:PinHeader_2x03_P2.00mm_Vertical, F.Cu at (171.7, 130.1)
- added J3: Barrel_Jack, Connector_BarrelJack:BarrelJack_CUI_PJ-063AH_Horizontal_CircularHoles, F.Cu at (178.3, 140.3)
- added R1: 1M, Resistor_SMD:R_0402_1005Metric, F.Cu at (221.8, 118.2)
- added R2: 1M, Resistor_SMD:R_0402_1005Metric, F.Cu at (163.4, 106.5)
- added U2: ATmega16U2-A, Package_QFP:TQFP-32_7x7mm_P0.8mm, F.Cu at (221.3, 136.5)
- added U3: LP2985-3.3, Package_TO_SOT_SMD:SOT-23-5, F.Cu at (181.0, 125.5)
- added U4: NCP1117-12_TO252, Package_TO_SOT_SMD:TO-252-2, F.Cu at (203.5, 112.8)
- added U5: RP2040, Package_DFN_QFN:QFN-56-1EP_7x7mm_P0.4mm_EP3.2x3.2mm, F.Cu at (177.5, 113.5)
- added Y2: Crystal, Crystal:Crystal_HC49-4H_Vertical, F.Cu at (219.0, 125.5)
- moved C1 67.3 mm to (218.3, 118.2)
- moved C2 66.5 mm to (225.9, 118.2)
- moved Y1 40.7 mm to (160.9, 113.6)
- moved U1 39.4 mm to (162.9, 122.8)
- moved J1 9.60 mm to (190.3, 147.7)

Commit message: massive gains
Parts:
- removed U5: RP2040, Package_DFN_QFN:QFN-56-1EP_7x7mm_P0.4mm_EP3.2x3.2mm
- removed Y1: Crystal, Crystal:Crystal_HC49-4H_Vertical
- added C10: 100nF, Capacitor_SMD:C_0402_1005Metric, F.Cu at (181.0, 54.9)
- added C11: 100nF, Capacitor_SMD:C_0402_1005Metric, F.Cu at (196.0, 54.1)
- added C12: 100nF, Capacitor_SMD:C_0402_1005Metric, F.Cu at (192.1, 44.7)
- added C5: 100nF, Capacitor_SMD:C_0402_1005Metric, F.Cu at (195.4, 100.5)
- added C6: 1uF, Capacitor_SMD:C_0402_1005Metric, F.Cu at (189.8, 107.9)
- added C7: 100nF, Capacitor_SMD:C_0402_1005Metric, F.Cu at (176.4, 97.7)
- added C8: 22uF, Capacitor_SMD:C_0402_1005Metric, F.Cu at (182.6, 93.7)
- added C9: 1uF, Capacitor_SMD:C_0402_1005Metric, F.Cu at (188.0, 59.4)
- added D1: Rst_D, Diode_SMD:D_SOD-323, B.Cu at (178.3, 47.8)
- added F1: MF-MSMF050-2, Fuse:Fuse_1812_4532Metric, F.Cu at (180.5, 96.8)
- added J4: Digital_Pins, Connector_PinHeader_2.54mm:PinHeader_1x17_P2.54mm_Vertical, F.Cu at (163.6, 79.8)
- added J5: Analog, Connector_PinHeader_2.54mm:PinHeader_1x06_P2.54mm_Vertical, F.Cu at (153.8, 80.8)
- added LED_BUILTIN1: green, LED_SMD:LED_0603_1608Metric, F.Cu at (178.3, 139.3)
- added ON1: blue, LED_SMD:LED_0603_1608Metric, F.Cu at (175.4, 139.3)
- added Q1: FDN340P, Package_TO_SOT_SMD:SOT-23, F.Cu at (180.3, 101.1)
- added R10: 10k, Resistor_SMD:R_0402_1005Metric, F.Cu at (197.7, 55.4)
- added R11: 10k, Resistor_SMD:R_0402_1005Metric, F.Cu at (183.9, 44.8)
- added R3: 10k, Resistor_SMD:R_0402_1005Metric, F.Cu at (176.4, 99.0)
- added R4: 22, Resistor_SMD:R_0402_1005Metric, F.Cu at (174.0, 64.9)
- added R5: 1k, Resistor_SMD:R_0402_1005Metric, F.Cu at (181.3, 136.6)
- added R6: 22, Resistor_SMD:R_0402_1005Metric, F.Cu at (174.0, 63.9)
- added R7: 1k, Resistor_SMD:R_0402_1005Metric, F.Cu at (184.2, 136.7)
- added R8: 1k, Resistor_SMD:R_0402_1005Metric, F.Cu at (178.3, 136.4)
- added R9: 1k, Resistor_SMD:R_0402_1005Metric, F.Cu at (175.4, 136.4)
- added RX1: yellow, LED_SMD:LED_0603_1608Metric, F.Cu at (181.3, 139.4)
- added SW1: Reset, Button_Switch_SMD:SW_SPST_TL3342, B.Cu at (174.8, 53.1)
- added TX1: yellow, LED_SMD:LED_0603_1608Metric, F.Cu at (184.2, 139.4)
- C1: value C -> 100nF
- C2: value C -> 22uF
- C3, C4: value C -> 22pF
- J1: value USB_B_Micro -> ISCP_CON; footprint Connector_USB:USB_Micro-B_Amphenol_10103594-0001LF_Horizontal -> Connector_PinHeader_2.54mm:PinHeader_2x03_P2.54mm_Vertical
- J2: value Conn_02x03_Counter_Clockwise_MountingPin -> USB_B_Micro; footprint Connector_PinHeader_2.00mm:PinHeader_2x03_P2.00mm_Vertical -> Connector_USB:USB_Micro-B_Molex-105017-0001
- J3: value Barrel_Jack -> Cons; footprint Connector_BarrelJack:BarrelJack_CUI_PJ-063AH_Horizontal_CircularHoles -> Connector_PinHeader_2.54mm:PinHeader_1x09_P2.54mm_Vertical
- R1: value 1M -> 10k
- U1: value ATmega328P-A -> ATmega32U4-A; footprint Package_QFP:TQFP-32_7x7mm_P0.8mm -> Package_QFP:TQFP-44_10x10mm_P0.8mm
- U2: value ATmega16U2-A -> PMV48XP_215; footprint Package_QFP:TQFP-32_7x7mm_P0.8mm -> footprints:TO-236_SOT23_NEX
- U3: value LP2985-3.3 -> NCP1117-5.0_SOT223; footprint Package_TO_SOT_SMD:SOT-23-5 -> Package_TO_SOT_SMD:SOT-223-3_TabPin2
- U4: value NCP1117-12_TO252 -> LP2985-3.3; footprint Package_TO_SOT_SMD:TO-252-2 -> Package_TO_SOT_SMD:SOT-23-5
- Y2: value Crystal -> 16MHz
- moved J1 104.5 mm to (201.8, 43.8), turned to 90 degrees
- moved U1 75.1 mm to (188.4, 52.1), turned to 90 degrees
- moved Y2 71.4 mm to (207.1, 55.1), turned to 90 degrees
- moved C3 67.6 mm to (203.6, 55.4), turned to 90 degrees
- moved R2 66.5 mm to (203.2, 53.2), turned to 90 degrees
- moved C4 66.4 mm to (203.5, 51.0), turned to -90 degrees
- moved J2 65.3 mm to (169.8, 64.8), turned to -90 degrees
- moved G*** 64.2 mm to (220.6, 115.8)
- moved U2 53.0 mm to (189.3, 94.2)
- moved J3 48.0 mm to (153.8, 99.1)
- moved R1 42.9 mm to (181.3, 104.2), turned to -90 degrees
- moved C2 36.2 mm to (194.3, 100.5), turned to -90 degrees
- moved C1 34.3 mm to (192.3, 95.9), turned to 90 degrees
- moved U3 26.1 mm to (188.5, 100.5), turned to 180 degrees
- moved U4 17.3 mm to (187.3, 106.6), turned to -90 degrees
Connections:
- C1 pad 1: GND -> Net-(U2-S)
- C1 pad 2: CLKA -> GND
- C2 pad 1: GND -> +5V
- C2 pad 2: CLKB -> GND
- C3 pad 2: CLKC -> XTAL2
- C4 pad 2: CLKD -> XTAL1
- J1 pad 1: unconnected-(J1-VBUS-Pad1) -> MISO
- J1 pad 2: unconnected-(J1-D--Pad2) -> +5V
- J1 pad 3: unconnected-(J1-D+-Pad3) -> SCK
- J1 pad 4: unconnected-(J1-ID-Pad4) -> MOSI
- J1 pad 5: unconnected-(J1-GND-Pad5) -> RESET
- J1 pad 6: unconnected-(J1-Shield-Pad6) -> GND
- J2 pad 1: unconnected-(J2-Pin_1-Pad1) -> Net-(J2-VBUS)
- J2 pad 2: unconnected-(J2-Pin_2-Pad2) -> Net-(J2-D-)
- J2 pad 3: unconnected-(J2-Pin_3-Pad3) -> Net-(J2-D+)
- J2 pad 5: unconnected-(J2-Pin_5-Pad5) -> GND
- J2 pad 6: unconnected-(J2-Pin_6-Pad6) -> GND
- J3 pad 1: unconnected-(J3-Pad1) -> ~IO13
- J3 pad 2: unconnected-(J3-Pad2) -> +3.3V
- R1 pad 1: CLKA -> Vin
- R1 pad 2: CLKB -> GND
- R2 pad 1: CLKC -> XTAL2
- R2 pad 2: CLKD -> XTAL1
- U1 pad 1: unconnected-(U1-PD3-Pad1) -> ~D7
- U1 pad 10: unconnected-(U1-PD6-Pad10) -> MOSI
- U1 pad 11: unconnected-(U1-PD7-Pad11) -> MISO
- U1 pad 12: unconnected-(U1-PB0-Pad12) -> ~IO11
- U1 pad 13: unconnected-(U1-PB1-Pad13) -> RST
- U1 pad 14: unconnected-(U1-PB2-Pad14) -> +5V
- U1 pad 15: unconnected-(U1-PB3-Pad15) -> GND
- U1 pad 16: unconnected-(U1-PB4-Pad16) -> XTAL2
- U1 pad 17: unconnected-(U1-PB5-Pad17) -> XTAL1
- U1 pad 18: unconnected-(U1-AVCC-Pad18) -> D3/SCL
- U1 pad 19: unconnected-(U1-ADC6-Pad19) -> D2/SDA
- U1 pad 2: unconnected-(U1-PD4-Pad2) -> +5V
- U1 pad 20: unconnected-(U1-AREF-Pad20) -> D0/RX
- U1 pad 21: Net-(U1-GND-Pad21) -> D1/TX
- U1 pad 22: unconnected-(U1-ADC7-Pad22) -> Net-(U1-PD5)
- U1 pad 23: unconnected-(U1-PC0-Pad23) -> GND
- U1 pad 24: unconnected-(U1-PC1-Pad24) -> +5V
- U1 pad 25: unconnected-(U1-PC2-Pad25) -> ~D4
- U1 pad 26: unconnected-(U1-PC3-Pad26) -> ~IO12
- U1 pad 27: unconnected-(U1-PC4-Pad27) -> ~D6
- U1 pad 28: unconnected-(U1-PC5-Pad28) -> IO8
- U1 pad 29: unconnected-(U1-~{RESET}/PC6-Pad29) -> ~IO9
- U1 pad 3: Net-(U1-GND-Pad21) -> D-
- U1 pad 30: unconnected-(U1-PD0-Pad30) -> ~IO10
- U1 pad 31: unconnected-(U1-PD1-Pad31) -> ~D5
- U1 pad 32: unconnected-(U1-PD2-Pad32) -> ~IO13
- U1 pad 4: Net-(U1-VCC-Pad4) -> D+
- U1 pad 5: Net-(U1-GND-Pad21) -> GND
- U1 pad 6: Net-(U1-VCC-Pad4) -> Net-(U1-UCAP)
- U1 pad 7: unconnected-(U1-XTAL1/PB6-Pad7) -> Vusb
- U1 pad 8: unconnected-(U1-XTAL2/PB7-Pad8) -> RX_LED
- U1 pad 9: unconnected-(U1-PD5-Pad9) -> SCK
- U2 pad 1: unconnected-(U2-XTAL1-Pad1) -> +5V
- U2 pad 2: unconnected-(U2-PC0/XTAL2-Pad2) -> Net-(U2-S)
- U2 pad 3: unconnected-(U2-GND-Pad3) -> Vin
- U3 pad 1: unconnected-(U3-VIN-Pad1) -> GND
- U3 pad 2: unconnected-(U3-GND-Pad2) -> +5V
- U3 pad 3: unconnected-(U3-ON/~{OFF}-Pad3) -> Net-(U2-S)
- U4 pad 1: GND -> +5V
- U4 pad 2: +5V -> GND
- U4 pad 3: Net-(U4-VI) -> +5V
Routing:
- net GND: track 0.00 -> 314.1 mm, vias 0 -> 1
- net +5V: track 0.00 -> 225.4 mm, vias 0 -> 5
- net MISO: track 0.00 -> 157.8 mm
- net MOSI: track 0.00 -> 139.0 mm, vias 0 -> 1
- net ~IO13: track 0.00 -> 127.3 mm
- net RST: track 0.00 -> 114.9 mm, vias 0 -> 1
- net SCK: track 0.00 -> 112.1 mm, vias 0 -> 1
- net Net-(U1-PD5): track 0.00 -> 102.3 mm, vias 0 -> 2
- net RX_LED: track 0.00 -> 101.9 mm, vias 0 -> 1
- net D0/RX: track 0.00 -> 88.3 mm, vias 0 -> 1
- net D1/TX: track 0.00 -> 81.5 mm, vias 0 -> 2
- net D2/SDA: track 0.00 -> 71.3 mm, vias 0 -> 2
- net ~D4: track 0.00 -> 65.2 mm, vias 0 -> 1
- net D3/SCL: track 0.00 -> 65.0 mm, vias 0 -> 1
- net AREF: track 0.00 -> 63.6 mm
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Other:
- board text added: "11/08/2023"
- board text added: "Amogduino REV 1.0"
- board text added: "JLCJLCJLCJLC"
- board text added: "LED"
- board text added: "https://github.com/AndrewMcGhee"
